File: pcbs/limbatus.kicad_pcb (KiCad board)
At the start: 2 copper layers, 249.5 x 112.1 mm, 78 parts

Commit message: Resync outlines/pcbs to config; define gerbers as production snapshots
main went red because outlines/pcbs committed in 00dc192 were regenerated
from an older config and never refreshed after the power-switch reposition,
GND stitching vias, and logo/silk changes landed. The Reproducibility job
correctly caught the drift.

Fix and policy:
- Regenerate outlines/pcbs from the current config so they match again and
  the Reproducibility gate passes. These artifacts track current design and
  must be committed alongside any config change (the gate enforces this).
- Define gerbers/ as PRODUCTION snapshots, decoupled from live outputs: only
  refreshed and committed when placing a physical fab order, tagged per run,
  with provenance in gerbers/SOURCE.md. They intentionally lag outlines/pcbs
  between orders and agree with them only at a fab tag. CI never regenerates
  or auto-commits gerbers.
- Document both policies in CLAUDE.md; add gerbers/SOURCE.md recording the
  current gerbers as a pre-production placeholder (not yet ordered).

Co-Authored-By: Claude Opus 4.8 <noreply@anthropic.com>
Parts:
- added LOGO1: , ceoloide:utility_ergogen_logo, B.Cu at (0.00, -6.00)
- added V1: , local:stitching_via, F.Cu at (0.00, -12.0)
- added V2: , local:stitching_via, F.Cu at (0.00, -18.0)
- added V3: , local:stitching_via, F.Cu at (-40.0, -80.0)
- added V4: , local:stitching_via, F.Cu at (-75.0, -80.0)
- added V5: , local:stitching_via, F.Cu at (-117.0, -37.0)
- added V6: , local:stitching_via, F.Cu at (40.0, -80.0)
- added V7: , local:stitching_via, F.Cu at (75.0, -80.0)
- added V8: , local:stitching_via, F.Cu at (117.0, -37.0)
- moved PWR1 36.0 mm to (-122.5, -60.5), turned to 180 degrees
Other:
- board text added: "JLCJLCJLCJLCJLCJLCJLC"
- board text added: "limbatus"
- board text added: "rev A 2026-07"
