File: production/2026-07-06-prototype/limbatus.kicad_pcb (KiCad board)
At the start: 2 copper layers, 249.5 x 112.1 mm, 87 parts

Commit message: Commit only production artifacts; stop committing live build outputs
Reframe what lives in git: ergogen/config.yaml is the source of truth, and the
only committed fabrication artifacts are frozen production bundles — never the
live, regenerable outputs.

- Gitignore and untrack the live build products: root outlines/, pcbs/, and
  gerbers/. Regenerate them with `make build` or pull the Build workflow's
  artifacts. This removes the whole class of "committed outputs drift from
  config" failures (stale artifacts, the daily date-stamp churn) at the root.
- Add production/ for immutable per-order bundles: gerbers + the matching
  limbatus.kicad_pcb + outlines + SOURCE.md provenance, tagged fab-<order-id>.
  Bundles are cut and committed by hand when ordering; CI never writes here.
- Preserve the existing (never-ordered) gerbers as production/2026-07-06-prototype,
  pairing them with the matching pcb/outlines from their source commit 00dc192
  so the bundle is internally consistent, clearly labeled not-yet-ordered.
- Remove the Reproducibility CI job (nothing left to diff against config).
  Build-success is still covered by the kibot and generate jobs.
- Document the model in CLAUDE.md and production/README.md.

Co-Authored-By: Claude Opus 4.8 <noreply@anthropic.com>
Parts:
- removed LOGO1: , ceoloide:utility_ergogen_logo
- removed V1, V2, V3, V4, V5, V6, V7, V8: , local:stitching_via
- moved PWR1 36.0 mm to (-97.7, -86.6), turned to 90 degrees
Other:
- board text removed: "JLCJLCJLCJLCJLCJLCJLC"
- board text removed: "limbatus"
- board text removed: "rev A 2026-07"
